File: xblast-lite.kicad_sch (KiCad schematic)
At the start: 12 parts, among them J1 TC2050, J2 LPC, J3 GPIO, J4 LCD, U1 74LVC125, U2 SST49LF080A-33-4C-NHE, U3 XC9572XL-xxVQx44, U4 TPS27081A

Commit message: WIP
Parts:
- added J5: PLCC-32 Socket, xblast-lite:PLCC-32_SMD-Socket, symbol Connector:Conn_01x32_Socket
- J2: value LPC -> XBOX LPC; footprint (none) -> Connector_PinSocket_2.54mm:PinSocket_2x06_P2.54mm_Vertical; Distributor Link 1 (none) -> https://www.digikey.com/en/products/detail/te-connectivity-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; Distributor Link 2 (none) -> https://www.mouser.com/en/ProductDetail/TE-Connectivity/5-5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; LCSC (none) -> C18078145; Manufacturer (none) -> Bossie; Manufacturer Part Number (none) -> BX-PM2.54-2-6PY
- U2: footprint (none) -> Package_LCC:PLCC-32_11.4x14.0mm_P1.27mm
Other:
- company: (none) -> Clegg
- title: (none) -> Xblast Lite
- moved on the sheet: J2, JP1, U2
Changed lines of the file:
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@@
 	(generator_version "10.0")
 	(paper "A4")
+	(title_block
+		(title "Xblast Lite")
+		(date "2026-09-17")
+		(rev "A")
+		(company "Clegg")
+	)

Commit message: WIP
Parts:
- added R1, R2: 10k, Resistor_SMD:R_0603_1608Metric, symbol Device:R_Small
- J4: footprint Connector_Molex:Molex_CLIK-Mate_502386-1170_1x11-1MP_P1.25mm_Horizontal -> Connector_JST:JST_XH_S12B-XH-A-1_1x12_P2.50mm_Horizontal; Distributor Link 1 (none) -> https://www.digikey.com/en/products/detail/jst-sales-americ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; Distributor Link 2 (none) -> https://www.mouser.com/en/ProductDetail/JST-Commercial/S12B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; LCSC (none) -> C566191; Manufacturer (none) -> JST; Manufacturer Part Number (none) -> S12B-XH-A-1
- J5: Distributor Link 1 (none) -> https://www.digikey.com/en/products/detail/assmann-wsw-comp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; LCSC (none) -> C6486301; Manufacturer (none) -> Assmann WSW Components; Manufacturer Part Number (none) -> A-CCS 032-Z-SM
- JP1: value Bank Switch -> Bank Lock; footprint Connector_PinSocket_2.54mm:PinSocket_1x03_P2.54mm_Vertical -> Jumper:SolderJumper-3_P1.3mm_Open_Pad1.0x1.5mm; symbol Jumper:Jumper_3_Open -> Jumper:SolderJumper_3_Open
Connections:
- net +5V_SUPPLY: now reaches U4.1 (R2)
- net +5V_SUPPLY: now also U4.2 (VOUT), U4.3 (VOUT)
- net +5V_LPC: now reaches U4.4 (VIN)
- net +5V_LPC: now also J2.6 (Pin_6), R1.2
- net EN_5V: now reaches U4.5 (ON/OFF)
- net EN_5V: now also R2.2
- net LDO_R1: now reaches U4.6 (R1/C1)
- net LDO_R1: now also R1.1
- net XLCLK: now reaches J2.1 (Pin_1)
- net XLAD1: now reaches J2.10 (Pin_10)
- net XLAD0: now reaches J2.11 (Pin_11)
- net GND: now reaches J2.12 (Pin_12)
- net GND: now also J2.2 (Pin_2), JP1.2 (C), R2.1
- net ~{XLFRAME}: now reaches J2.3 (Pin_3)
- net ~{XLRESET}: now reaches J2.5 (Pin_5)
- net XLAD3: now reaches J2.7 (Pin_7)
- net XLAD2: now reaches J2.8 (Pin_8)
- net +3V3: now reaches J2.9 (Pin_9)
- net BANK_SW0: now reaches JP1.1 (A)
- net BANK_SW1: now reaches JP1.3 (B)
- no-connect marks 0 -> 1
