File: xblast-lite.kicad_sch (KiCad schematic)
At the start: 31 parts, among them J1 TC2050, J2 XBOX LPC, J3 GPIO, J4 LCD, J5 PLCC-32 Socket, Q1 BC846, Q2 BC846, U1 74LVC125, U2 SST49LF080A-33-4C-NHE, U3 XC9572XL-xxVQx44, U4 TPS27081A

Commit message: Finished layout
Parts:
- J1: value TC2050 -> JTAG
